File: pcb/adelheid.kicad_pcb (KiCad board)
At the start: 2 copper layers, 339.1 x 142.6 mm, 206 parts, among them J1 USB_B_Mini, J10 PF6, J11 PF4, J12 VCC, J13 D+, J14 D-, J15 GND, J2 MISO, J3 VCC, J4 SCK, J5 MOSI, J6 RES, J7 GND, J9 PF5, SW0 SW_Push, SW1 SW_Push, SW10 SW_Push, SW11 SW_Push, SW12 SW_Push, SW13 SW_Push, SW14 SW_Push, SW15 SW_Push, SW16 SW_Push, SW17 SW_Push, SW18 SW_Push, SW19 SW_Push, SW2 SW_Push, SW20 SW_Push, SW21 SW_Push, SW22 SW_Push, SW23 SW_Push, SW24 SW_Push, SW25 SW_Push, SW26 SW_Push, SW27 SW_Push, SW28 SW_Push, SW29 SW_Push, SW3 SW_Push, SW30 SW_Push, SW31 SW_Push, SW32 SW_Push, SW33 SW_Push, SW34 SW_Push, SW35 SW_Push, SW36 SW_Push, SW37 SW_Push, SW38 SW_Push, SW39 SW_Push, SW3s1 SW_Push, SW4 SW_Push, SW40 SW_Push, SW41 SW_Push, SW42 SW_Push, SW43 SW_Push, SW44 SW_Push, SW45 SW_Push, SW46 SW_Push, SW47 SW_Push, SW48 SW_Push, SW49 SW_Push, SW5 SW_Push, SW50 SW_Push, SW51 SW_Push, SW52 SW_Push, SW53 SW_Push, SW54 SW_Push, SW55 SW_Push, SW56 SW_Push, SW57 SW_Push, SW58 SW_Push, SW59 SW_Push, SW6 SW_Push, SW60 SW_Push, SW61 SW_Push, SW62 SW_Push, SW63 SW_Push, SW64 SW_Push, SW65 SW_Push, SW66 SW_Push, SW67 SW_Push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

Commit message: updated pcb labels to be more consistent [v1.0.1]
Parts:
- J1: value USB_B_Mini -> J1
- moved D32 23.6 mm to (198.9, 137.2)
- moved D41 23.6 mm to (236.1, 129.3)
- moved SW33 23.6 mm to (162.9, 150.0)
- moved D1 23.6 mm to (43.9, 66.1)
- moved D38 23.6 mm to (205.7, 77.3)
- moved D55 23.6 mm to (281.2, 66.1)
- moved D59 23.6 mm to (300.2, 66.1)
- moved D6 23.6 mm to (62.9, 66.1)
- moved D63 23.6 mm to (319.3, 66.1)
- moved H1 23.6 mm to (56.6, 71.9)
- moved H7 23.6 mm to (340.9, 67.1)
- moved C5 23.6 mm to (165.7, 36.0)
- moved C6 23.6 mm to (165.7, 38.0)
- moved C7 23.6 mm to (180.6, 49.9)
- moved C8 23.6 mm to (164.9, 45.5)
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- renumbered SW9 to SW10, SW69 to SW11, SW10 to SW12, SW11 to SW13, SW12 to SW14, SW13 to SW15, SW14 to SW16, SW70 to SW17, SW15 to SW18, SW16 to SW19, SW17 to SW20, SW18 to SW21, SW71 to SW22, SW19 to SW23, SW20 to SW24, SW21 to SW25, SW22 to SW26, SW23 to SW27, SW72 to SW28, SW24 to SW29, SW25 to SW30, SW26 to SW31, SW27 to SW32, SW28 to SW33, SW73 to SW34, SW29 to SW35, SW30 to SW36, SW31 to SW37, SW32 to SW38, SW74 to SW39, SW33 to SW40, SW34 to SW41, SW35 to SW42, SW36 to SW43, SW37 to SW44, SW75 to SW45, SW38 to SW46, SW39 to SW47, SW40 to SW48, SW41 to SW49, SW76 to SW50, SW42 to SW51, SW43 to SW52, SW44 to SW53, SW45 to SW54, SW46 to SW55, SW77 to SW56, SW47 to SW57, SW48 to SW58, SW49 to SW59, SW68 to SW6, SW50 to SW60, SW78 to SW61, SW51 to SW62, SW52 to SW63, SW53 to SW64, SW54 to SW65, SW79 to SW66, SW55 to SW67, SW56 to SW68, SW57 to SW69, SW6 to SW7, SW58 to SW70, SW80 to SW71, SW59 to SW72, SW60 to SW73, SW61 to SW74, SW62 to SW75, SW81 to SW76, SW63 to SW77, SW64 to SW78, SW65 to SW79, SW7 to SW8, SW66 to SW80, SW67 to SW81, SW8 to SW9
Other:
- board text added: "fork of FateNozomi/Arisu by floookay [v1.0.1]"
- board text added: "•"
- board text removed: "fork of FateNozomi/Arisu by floookay [v1]"
