File: pcb/adelheid.kicad_pcb (KiCad board)
At the start: 2 copper layers, 339.1 x 143.2 mm, 323 parts, among them J1 USB_B_Mini, J12 VCC, J13 D+, J14 D-, J15 GND, J2 MISO, J3 VCC, J4 SCK, J5 MOSI, J6 RES, J7 GND, J8 PF4, J9 PF5, Q1 2N7002, U1 USBLC6-2SC6, U2 ATmega32U4-AU, Y1 Crystal_GND24

Commit message: fixed revision number [Rev1.0]
Other:
- board text added: "fork of FateNozomi/arisu-pcb by floookay [Rev1.0]"
- board text removed: "fork of FateNozomi/arisu-pcb by floookay [v2]"
Changed lines of the file:
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@@
   (title_block
     (title "Adelheid")
-    (rev "2.0")
+    (rev "1.0")
     (company "floookay")
   )
@@
     (effects (font (size 1.5 1.5) (thickness 0.375)))
   )
-  (gr_text "fork of FateNozomi/arisu-pcb\nby floookay [v2]" (at 287.147 146.177) (layer "B.SilkS")
+  (gr_text "fork of FateNozomi/arisu-pcb\nby floookay [Rev1.0]" (at 287.147 146.177) (layer "B.SilkS")
     (effects (font (size 1.5 1.5) (thickness 0.3)) (justify mirror))
   )
