File: pcb/adelheid.sch (KiCad schematic (older format))
At the start: 40 parts, among them J1 USB_B_Micro, J10 PF6, J11 PF7, J12 VCC, J13 D+, J14 D-, J15 GND, J2 MISO, J3 VCC, J4 SCK, J5 MOSI, J6 RES, J7 GND, J8 PF4, J9 PF5, U1 USBLC6-2SC6, U2 ATmega32U4-AU, Y1 Crystal_GND24

Commit message: initial commit
Parts:
- removed J1: USB_B_Micro, Connectors_USB:USB_Micro-B_Molex-105017-0001, symbol Connector:USB_B_Micro
- removed J8: PF4, Pin_Headers:Pin_Header_Straight_1x01_Pitch2.54mm, symbol Connector_Generic:Conn_01x01
- added J1: USB_B_Mini, Keebio-Parts:USB-Mini-B_2leg, symbol Connector:USB_B_Mini
- C1, C2: LCSC (none) -> C1804
- C3: LCSC (none) -> C15850
- C4, C5: LCSC (none) -> C28323
- C6, C7, C8, C9: LCSC (none) -> C49678
- J11: value PF7 -> PF4
- U2: symbol MCU_Microchip_ATmega:ATmega32U4-AU -> adelheid-rescue:ATmega32U4-AU-MCU_Microchip_ATmega-arisu-rescue
Connections:
- net labels added: row00
- net labels removed: PF7
- wire segments 131 -> 135
Other:
- moved on the sheet: J11
