File: pcb/adelheid.sch (KiCad schematic (older format))
At the start: 40 parts, among them J1 USB_B_Mini, J12 VCC, J13 D+, J14 D-, J15 GND, J2 MISO, J3 VCC, J4 SCK, J5 MOSI, J6 RES, J7 GND, J8 PF4, J9 PF5, Q1 2N7002, U1 USBLC6-2SC6, U2 ATmega32U4-AU, Y1 Crystal_GND24

Commit message: restructured folder structure
Parts:
- U2: symbol arisu-rescue:ATmega32U4-AU-MCU_Microchip_ATmega -> adelheid-rescue:ATmega32U4-AU-MCU_Microchip_ATmega
Changed lines of the file:
@@
 $EndDescr
 $Comp
-L arisu-rescue:ATmega32U4-AU-MCU_Microchip_ATmega U2
+L adelheid-rescue:ATmega32U4-AU-MCU_Microchip_ATmega U2
 U 1 1 5C4B1F82
 P 4500 4250

Commit message: switched backlight pin [Rev2.0]
swapped col4 and led pin.
Backlight is now on pin 31 (C6).
In Rev1.0 the backlight started flickering because the MCU couldn't
handle the load of the LEDs on pin 37. This should fix the issue.
Thank you u/SryImBadAtNaming for finding out and notifying me!
Parts:
- U1: symbol Power_Protection:USBLC6-2SC6 -> adelheid-rescue:USBLC6-2SC6-Power_Protection
Connections:
- net col4: now also U2.37 (PF6); no longer U2.31 (PC6)
- net at R5.1: now also U2.31 (PC6); no longer U2.37 (PF6)
Other:
- moved on the sheet: R5
Changed lines of the file:
@@
-EESchema Schematic File Version 5
+EESchema Schematic File Version 4
 EELAYER 30 0
 EELAYER END
@@
 Title "Adelheid"
 Date ""
-Rev "1.0"
+Rev "2.0"
 Comp "floookay"
 Comment1 ""
@@
 Comment3 ""
 Comment4 ""
-Comment5 ""
-Comment6 ""
-Comment7 ""
-Comment8 ""
-Comment9 ""
 $EndDescr
 $Comp
@@
 $EndComp
 $Comp
-L Power_Protection:USBLC6-2SC6 U1
+L adelheid-rescue:USBLC6-2SC6-Power_Protection U1
 U 1 1 5C4B2347
 P 1900 5650
@@
 	5100 3450 6650 3450
 Wire Wire Line
-	5100 3650 6650 3650
-Wire Wire Line
 	5100 3750 6650 3750
 Wire Wire Line
@@
 Wire Wire Line
 	6450 5650 6450 5750
-Wire Wire Line
-	6100 5950 6150 5950
 $Comp
 L power:GND #PWR0122
@@
 L Device:R R5
 U 1 1 5EC25C97
-P 5950 5550
-F 0 "R5" V 6050 5500 50  0000 L CNN
-F 1 "1.5K" V 5950 5450 46  0000 L CNN
-F 2 "Resistor_SMD:R_0805_2012Metric_Pad1.15x1.40mm_HandSolder" V 5880 5550 50  0001 C CNN
-F 3 "~" H 5950 5550 50  0001 C CNN
-	1    5950 5550
+P 5600 3650
+F 0 "R5" V 5700 3600 50  0000 L CNN
+F 1 "1.5K" V 5600 3550 46  0000 L CNN
+F 2 "Resistor_SMD:R_0805_2012Metric_Pad1.15x1.40mm_HandSolder" V 5530 3650 50  0001 C CNN
+F 3 "~" H 5600 3650 50  0001 C CNN
+	1    5600 3650
 	0    -1   -1   0
 $EndComp
 Wire Wire Line
-	6100 5550 6100 5950
-Wire Wire Line
-	5100 5550 5800 5550
-Wire Wire Line
 	6200 5350 6200 5650
 Wire Wire Line
 	5100 5650 6200 5650
+Wire Wire Line
+	5100 3650 5450 3650
+Wire Wire Line
+	5750 3650 6000 3650
+Wire Wire Line
+	6000 3650 6000 5950
+Wire Wire Line
+	6000 5950 6150 5950
+Wire Wire Line
+	5100 5550 6150 5550
+Wire Wire Line
+	6150 5550 6150 3650
+Wire Wire Line
+	6150 3650 6650 3650
 Wire Bus Line
 	5750 2700 5750 3150
