File: arisu.kicad_pcb (KiCad board)
At the start: 2 copper layers, 339.1 x 118.7 mm, 176 parts, among them J1 USB_B_Micro, SW1 SW_Push, SW10 SW_Push, SW11 SW_Push, SW12 SW_Push, SW13 SW_Push, SW14 SW_Push, SW15 SW_Push, SW16 SW_Push, SW17 SW_Push, SW18 SW_Push, SW19 SW_Push, SW2 SW_Push, SW20 SW_Push, SW21 SW_Push, SW22 SW_Push, SW23 SW_Push, SW24 SW_Push, SW25 SW_Push, SW26 SW_Push, SW27 SW_Push, SW28 SW_Push, SW29 SW_Push, SW3 SW_Push, SW30 SW_Push, SW31 SW_Push, SW32 SW_Push, SW33 SW_Push, SW34 SW_Push, SW35 SW_Push, SW36 SW_Push, SW37 SW_Push, SW38 SW_Push, SW39 SW_Push, SW4 SW_Push, SW40 SW_Push, SW41 SW_Push, SW42 SW_Push, SW43 SW_Push, SW44 SW_Push, SW45 SW_Push, SW46 SW_Push, SW47 SW_Push, SW48 SW_Push, SW49 SW_Push, SW5 SW_Push, SW50 SW_Push, SW51 SW_Push, SW52 SW_Push, SW53 SW_Push, SW54 SW_Push, SW55 SW_Push, SW56 SW_Push, SW57 SW_Push, SW58 SW_Push, SW59 SW_Push, SW6 SW_Push, SW60 SW_Push, SW61 SW_Push, SW62 SW_Push, SW63 SW_Push, SW64 SW_Push, SW65 SW_Push, SW66 SW_Push, SW67 SW_Push, SW7 SW_Push, SW8 SW_Push, SW9 SW_Push, U1 USBLC6-2SC6, U2 ATmega32U4-AU, Y1 Crystal_GND24

Commit message: added footprints
Parts:
- removed G*** (x2): LOGO, arisu:arisu-logo
- removed PF6: PF6, Pin_Headers:Pin_Header_Straight_1x01_Pitch2.54mm
- removed PF7: PF7, Pin_Headers:Pin_Header_Straight_1x01_Pitch2.54mm
- removed SW1, SW10, SW11, SW12, SW13, SW15, SW16, SW17, SW18, SW19, SW20, SW21, SW22, SW24, SW25, SW26, SW27, SW28, SW29, SW30, SW31, SW32, SW33, SW34, SW35, SW36, SW38, SW39, SW40, SW41, SW42, SW43, SW44, SW45, SW47, SW48, SW49, SW50, SW51, SW52, SW53, SW55, SW56, SW58, SW59, SW6, SW61, SW62, SW63, SW64, SW65, SW66, SW67, SW7, SW8, SW9: SW_Push, Fate_Parts:SW_Cherry_MX_1.00u_PCB
- removed SW14, SW2, SW46, SW5, SW60: SW_Push, Fate_Parts:SW_Cherry_MX_1.50u_PCB
- removed SW23: SW_Push, Fate_Parts:SW_Cherry_MX_2.00u_PCB_ReversedStabilizers
- removed SW3, SW54: SW_Push, Fate_Parts:SW_Cherry_MX_1.75u_PCB
- removed SW37: SW_Push, Fate_Parts:SW_Cherry_MX_2.75u_PCB_ReversedStabilizers
- removed SW4: SW_Push, Fate_Parts:SW_Cherry_MX_2.25u_PCB
- removed SW57: SW_Push, Fate_Parts:SW_Cherry_MX_2.25u_PCB_ReversedStabilizers
- added D68: D, Diode_SMD:D_SOD-123, B.Cu at (291.9, 63.0)
- added D69: D, Diode_SMD:D_SOD-123, B.Cu at (305.6, 82.1)
- added D70: D, Diode_SMD:D_SOD-123, B.Cu at (326.5, 101.3)
- added D71: D, Diode_SMD:D_SOD-123, B.Cu at (324.2, 143.9)
- added D72: D, Diode_SMD:D_SOD-123, B.Cu at (323.6, 39.3)
- added D73: D, Diode_SMD:D_SOD-123, B.Cu at (311.0, 63.1)
- added D74: D, Diode_SMD:D_SOD-123, B.Cu at (329.4, 82.2)
- added D75: D, Diode_SMD:D_SOD-123, B.Cu at (343.3, 124.9)
- added D76: D, Diode_SMD:D_SOD-123, B.Cu at (343.2, 143.9)
- added D77: D, Diode_SMD:D_SOD-123, B.Cu at (349.6, 39.2)
- added D78: D, Diode_SMD:D_SOD-123, B.Cu at (330.1, 63.1)
- added D79: D, Diode_SMD:D_SOD-123, B.Cu at (353.9, 58.3)
- added D80: D, Diode_SMD:D_SOD-123, B.Cu at (358.1, 77.5)
- added D81: D, Diode_SMD:D_SOD-123, B.Cu at (362.2, 96.4)
- added D82: D, Diode_SMD:D_SOD-123, B.Cu at (362.3, 143.9)
- added MX1: MX-LED, ai03-MX_only:MXOnly-1U, F.Cu at (37.4, 39.3)
- added MX10: MX-LED, ai03-MX_only:MXOnly-1U, F.Cu at (72.5, 101.2)
- added MX11: MX-LED, ai03-MX_only:MXOnly-1U, F.Cu at (77.8, 120.2)
- added MX12: MX-LED, ai03-MX_only:MXOnly-1U, F.Cu at (80.4, 37.8)
- added MX13: MX-LED, ai03-MX_only:MXOnly-1U, F.Cu at (85.5, 61.6)
- added MX14: MX-LED, ai03-MX_only:MXOnly-1U, F.Cu at (92.3, 82.5)
- added MX15: MX-LED, ai03-MX_only:MXOnly-1U, F.Cu at (93.0, 102.1)
- added MX16: MX-LED, ai03-MX_only:MXOnly-1U, F.Cu at (98.3, 122.7)
- added MX17: MX-LED, ai03-MX_only:MXOnly-1.5U, F.Cu at (99.0, 142.3)
- added MX18: MX-LED, ai03-MX_only:MXOnly-1U, F.Cu at (101.2, 40.6)
- added MX19: MX-LED, ai03-MX_only:MXOnly-1U, F.Cu at (105.6, 65.8)
- added MX2: MX-LED, ai03-MX_only:MXOnly-1U, F.Cu at (47.4, 63.1)
- added MX20: MX-LED, ai03-MX_only:MXOnly-1U, F.Cu at (110.9, 86.4)
- added MX21: MX-LED, ai03-MX_only:MXOnly-1U, F.Cu at (111.6, 106.1)
- added MX22: MX-LED, ai03-MX_only:MXOnly-1U, F.Cu at (116.9, 126.7)
- added MX23: MX-LED, ai03-MX_only:MXOnly-1U, F.Cu at (119.8, 44.5)
- added MX24: MX-LED, ai03-MX_only:MXOnly-1U, F.Cu at (124.2, 69.8)
- added MX25: MX-LED, ai03-MX_only:MXOnly-1U, F.Cu at (129.5, 90.4)
- added MX26: MX-LED, ai03-MX_only:MXOnly-1U, F.Cu at (130.2, 110.0)
- added MX27: MX-LED, ai03-MX_only:MXOnly-1U, F.Cu at (135.6, 130.6)
- added MX28: MX-LED, ai03-MX_only:MXOnly-2U-FLIPPED-ReversedStabilizers, F.Cu at (131.6, 149.3)
- added MX29: MX-LED, ai03-MX_only:MXOnly-1U, F.Cu at (143.1, 49.5)
- added MX3: MX-LED, ai03-MX_only:MXOnly-1.5U, F.Cu at (48.0, 82.1)
- added MX30: MX-LED, ai03-MX_only:MXOnly-1U, F.Cu at (142.8, 73.7)
- added MX31: MX-LED, ai03-MX_only:MXOnly-1U, F.Cu at (148.2, 94.3)
- added MX32: MX-LED, ai03-MX_only:MXOnly-1U, F.Cu at (148.9, 114.0)
- added MX33: MX-LED, ai03-MX_only:MXOnly-1U, F.Cu at (154.2, 134.6)
- added MX34: MX-LED, ai03-MX_only:MXOnly-1U, F.Cu at (159.6, 155.2)
- added MX35: MX-LED, ai03-MX_only:MXOnly-1U, F.Cu at (161.7, 53.4)
- added MX36: MX-LED, ai03-MX_only:MXOnly-1U, F.Cu at (161.5, 77.7)
- added MX37: MX-LED, ai03-MX_only:MXOnly-1U, F.Cu at (184.3, 98.3)
- added MX38: MX-LED, ai03-MX_only:MXOnly-1U, F.Cu at (192.9, 115.9)
- added MX39: MX-LED, ai03-MX_only:MXOnly-1U, F.Cu at (201.5, 133.6)
- added MX4: MX-LED, ai03-MX_only:MXOnly-1.75U, F.Cu at (46.3, 101.2)
- added MX40: MX-LED, ai03-MX_only:MXOnly-1U, F.Cu at (189.3, 53.4)
- added MX41: MX-LED, ai03-MX_only:MXOnly-1U, F.Cu at (189.6, 77.7)
- added MX42: MX-LED, ai03-MX_only:MXOnly-1U, F.Cu at (202.9, 94.3)
- added MX43: MX-LED, ai03-MX_only:MXOnly-1U, F.Cu at (211.5, 112.0)
- added MX44: MX-LED, ai03-MX_only:MXOnly-1U, F.Cu at (220.1, 129.6)
- added MX45: MX-LED, ai03-MX_only:MXOnly-2.75U-ReversedStabilizers, F.Cu at (212.4, 150.7)
- added MX46: MX-LED, ai03-MX_only:MXOnly-1U, F.Cu at (207.9, 49.5)
- added MX47: MX-LED, ai03-MX_only:MXOnly-1U, F.Cu at (208.3, 73.7)
- added MX48: MX-LED, ai03-MX_only:MXOnly-1U, F.Cu at (221.5, 90.4)
- added MX49: MX-LED, ai03-MX_only:MXOnly-1U, F.Cu at (230.1, 108.0)
- added MX4_1: MX-LED, ai03-MX_only:MXOnly-1.75U-FLIPPED, F.Cu at (41.5, 101.2)
- added MX5: MX-LED, ai03-MX_only:MXOnly-2.25U, F.Cu at (46.9, 120.2)
- added MX50: MX-LED, ai03-MX_only:MXOnly-1U, F.Cu at (238.7, 125.7)
- added MX51: MX-LED, ai03-MX_only:MXOnly-1U, F.Cu at (231.2, 44.5)
- added MX52: MX-LED, ai03-MX_only:MXOnly-1U, F.Cu at (226.9, 69.8)
- added MX53: MX-LED, ai03-MX_only:MXOnly-1U, F.Cu at (240.1, 86.4)
- added MX54: MX-LED, ai03-MX_only:MXOnly-1U, F.Cu at (248.7, 104.1)
- added MX55: MX-LED, ai03-MX_only:MXOnly-1U, F.Cu at (257.4, 121.7)
- added MX56: MX-LED, ai03-MX_only:MXOnly-1.5U, F.Cu at (252.0, 142.3)
- added MX57: MX-LED, ai03-MX_only:MXOnly-1U, F.Cu at (249.9, 40.5)
- added MX58: MX-LED, ai03-MX_only:MXOnly-1U, F.Cu at (245.5, 65.8)
- added MX59: MX-LED, ai03-MX_only:MXOnly-1U, F.Cu at (258.8, 82.5)
- added MX6: MX-LED, ai03-MX_only:MXOnly-1.5U, F.Cu at (39.8, 139.3)
- added MX60: MX-LED, ai03-MX_only:MXOnly-1U, F.Cu at (269.2, 101.2)
- added MX61: MX-LED, ai03-MX_only:MXOnly-1U, F.Cu at (278.8, 120.2)
- added MX62: MX-LED, ai03-MX_only:MXOnly-1U, F.Cu at (270.6, 37.8)
- added MX63: MX-LED, ai03-MX_only:MXOnly-1U, F.Cu at (265.6, 61.6)
- added MX64: MX-LED, ai03-MX_only:MXOnly-1U, F.Cu at (279.3, 82.1)
- added MX65: MX-LED, ai03-MX_only:MXOnly-1U, F.Cu at (288.3, 101.2)
- added MX66: MX-LED, ai03-MX_only:MXOnly-1.75U, F.Cu at (305.0, 120.2)
- added MX67: MX-LED, ai03-MX_only:MXOnly-1U, F.Cu at (289.7, 37.8)
- added MX68: MX-LED, ai03-MX_only:MXOnly-1U, F.Cu at (284.6, 63.1)
- added MX69: MX-LED, ai03-MX_only:MXOnly-1U, F.Cu at (298.3, 82.1)
- added MX7: MX-LED, ai03-MX_only:MXOnly-1U, F.Cu at (61.4, 37.8)
- added MX70: MX-LED, ai03-MX_only:MXOnly-2.25U-FLIPPED-ReversedStabilizers, F.Cu at (319.2, 101.2)
- added MX71: MX-LED, ai03-MX_only:MXOnly-1U, F.Cu at (316.9, 144.0)
- added MX72: MX-LED, ai03-MX_only:MXOnly-1U, F.Cu at (316.3, 39.3)
- added MX73: MX-LED, ai03-MX_only:MXOnly-1U, F.Cu at (303.7, 63.1)
- added MX74: MX-LED, ai03-MX_only:MXOnly-1.5U, F.Cu at (322.1, 82.1)
- added MX75: MX-LED, ai03-MX_only:MXOnly-1U, F.Cu at (335.9, 125.0)
- added MX76: MX-LED, ai03-MX_only:MXOnly-1U, F.Cu at (335.9, 144.0)
- added MX77: MX-LED, ai03-MX_only:MXOnly-1U, F.Cu at (342.3, 39.3)
- added MX78: MX-LED, ai03-MX_only:MXOnly-1U, F.Cu at (322.7, 63.1)
- added MX79: MX-LED, ai03-MX_only:MXOnly-1U, F.Cu at (346.5, 58.3)
- added MX8: MX-LED, ai03-MX_only:MXOnly-1U, F.Cu at (66.4, 63.1)
- added MX80: MX-LED, ai03-MX_only:MXOnly-1U, F.Cu at (350.7, 77.4)
- added MX81: MX-LED, ai03-MX_only:MXOnly-1U, F.Cu at (355.0, 96.4)
- added MX82: MX-LED, ai03-MX_only:MXOnly-1U, F.Cu at (355.0, 144.0)
- added MX9: MX-LED, ai03-MX_only:MXOnly-1U, F.Cu at (71.8, 82.1)
- added Q1: 2N7002, Package_TO_SOT_SMD:SOT-23, B.Cu at (159.8, 37.3)
- added R5: 1.5K, Resistor_SMD:R_0805_2012Metric_Pad1.15x1.40mm_HandSolder, B.Cu at (155.9, 35.3)
- added RL1: R, Resistor_SMD:R_0805_2012Metric_Pad1.15x1.40mm_HandSolder, B.Cu at (44.7, 44.7)
- added RL10: R, Resistor_SMD:R_0805_2012Metric_Pad1.15x1.40mm_HandSolder, B.Cu at (79.8, 106.7)
- added RL11: R, Resistor_SMD:R_0805_2012Metric_Pad1.15x1.40mm_HandSolder, B.Cu at (85.1, 125.7)
- added RL12: R, Resistor_SMD:R_0805_2012Metric_Pad1.15x1.40mm_HandSolder, B.Cu at (87.6, 43.2)
- added RL13: R, Resistor_SMD:R_0805_2012Metric_Pad1.15x1.40mm_HandSolder, B.Cu at (92.7, 67.0)
- added RL14: R, Resistor_SMD:R_0805_2012Metric_Pad1.15x1.40mm_HandSolder, B.Cu at (98.3, 89.4)
- added RL15: R, Resistor_SMD:R_0805_2012Metric_Pad1.15x1.40mm_HandSolder, B.Cu at (99.1, 109.0)
- added RL16: R, Resistor_SMD:R_0805_2012Metric_Pad1.15x1.40mm_HandSolder, B.Cu at (104.4, 129.6)
- added RL17: R, Resistor_SMD:R_0805_2012Metric_Pad1.15x1.40mm_HandSolder, B.Cu at (105.2, 149.1)
- added RL18: R, Resistor_SMD:R_0805_2012Metric_Pad1.15x1.40mm_HandSolder, B.Cu at (107.3, 47.5)
- added RL19: R, Resistor_SMD:R_0805_2012Metric_Pad1.15x1.40mm_HandSolder, B.Cu at (111.5, 72.6)
- added RL2: R, Resistor_SMD:R_0805_2012Metric_Pad1.15x1.40mm_HandSolder, B.Cu at (54.7, 68.6)
- added RL20: R, Resistor_SMD:R_0805_2012Metric_Pad1.15x1.40mm_HandSolder, B.Cu at (116.8, 93.2)
- added RL21: R, Resistor_SMD:R_0805_2012Metric_Pad1.15x1.40mm_HandSolder, B.Cu at (117.6, 112.8)
- added RL22: R, Resistor_SMD:R_0805_2012Metric_Pad1.15x1.40mm_HandSolder, B.Cu at (122.9, 133.4)
- added RL23: R, Resistor_SMD:R_0805_2012Metric_Pad1.15x1.40mm_HandSolder, B.Cu at (125.9, 51.4)
- added RL24: R, Resistor_SMD:R_0805_2012Metric_Pad1.15x1.40mm_HandSolder, B.Cu at (130.3, 76.7)
- added RL25: R, Resistor_SMD:R_0805_2012Metric_Pad1.15x1.40mm_HandSolder, B.Cu at (135.6, 97.3)
- added RL26: R, Resistor_SMD:R_0805_2012Metric_Pad1.15x1.40mm_HandSolder, B.Cu at (136.2, 116.8)
- added RL27: R, Resistor_SMD:R_0805_2012Metric_Pad1.15x1.40mm_HandSolder, B.Cu at (141.4, 137.4)
- added RL28: R, Resistor_SMD:R_0805_2012Metric_Pad1.15x1.40mm_HandSolder, B.Cu at (137.6, 156.0)
- added RL29: R, Resistor_SMD:R_0805_2012Metric_Pad1.15x1.40mm_HandSolder, B.Cu at (149.1, 56.4)
- added RL3: R, Resistor_SMD:R_0805_2012Metric_Pad1.15x1.40mm_HandSolder, B.Cu at (55.1, 87.6)
- added RL30: R, Resistor_SMD:R_0805_2012Metric_Pad1.15x1.40mm_HandSolder, B.Cu at (148.8, 80.5)
- added RL31: R, Resistor_SMD:R_0805_2012Metric_Pad1.15x1.40mm_HandSolder, B.Cu at (154.2, 101.3)
- added RL32: R, Resistor_SMD:R_0805_2012Metric_Pad1.15x1.40mm_HandSolder, B.Cu at (154.9, 120.9)
- added RL33: R, Resistor_SMD:R_0805_2012Metric_Pad1.15x1.40mm_HandSolder, B.Cu at (160.1, 141.5)
- added RL34: R, Resistor_SMD:R_0805_2012Metric_Pad1.15x1.40mm_HandSolder, B.Cu at (165.6, 162.1)
- added RL35: R, Resistor_SMD:R_0805_2012Metric_Pad1.15x1.40mm_HandSolder, B.Cu at (165.4, 58.2)
- added RL36: R, Resistor_SMD:R_0805_2012Metric_Pad1.15x1.40mm_HandSolder, B.Cu at (167.6, 84.3)
- added RL37: R, Resistor_SMD:R_0805_2012Metric_Pad1.15x1.40mm_HandSolder, B.Cu at (192.6, 102.0)
- added RL38: R, Resistor_SMD:R_0805_2012Metric_Pad1.15x1.40mm_HandSolder, B.Cu at (201.1, 119.8)
- added RL39: R, Resistor_SMD:R_0805_2012Metric_Pad1.15x1.40mm_HandSolder, B.Cu at (209.8, 137.3)
- added RL4: R, Resistor_SMD:R_0805_2012Metric_Pad1.15x1.40mm_HandSolder, B.Cu at (53.6, 106.7)
- added RL40: R, Resistor_SMD:R_0805_2012Metric_Pad1.15x1.40mm_HandSolder, B.Cu at (197.8, 57.2)
- added RL41: R, Resistor_SMD:R_0805_2012Metric_Pad1.15x1.40mm_HandSolder, B.Cu at (197.9, 81.4)
- added RL42: R, Resistor_SMD:R_0805_2012Metric_Pad1.15x1.40mm_HandSolder, B.Cu at (211.2, 98.1)
- added RL43: R, Resistor_SMD:R_0805_2012Metric_Pad1.15x1.40mm_HandSolder, B.Cu at (219.8, 115.8)
- added RL44: R, Resistor_SMD:R_0805_2012Metric_Pad1.15x1.40mm_HandSolder, B.Cu at (228.4, 133.4)
- added RL45: R, Resistor_SMD:R_0805_2012Metric_Pad1.15x1.40mm_HandSolder, B.Cu at (220.8, 154.6)
- added RL46: R, Resistor_SMD:R_0805_2012Metric_Pad1.15x1.40mm_HandSolder, B.Cu at (216.2, 53.2)
- added RL47: R, Resistor_SMD:R_0805_2012Metric_Pad1.15x1.40mm_HandSolder, B.Cu at (216.4, 77.5)
- added RL48: R, Resistor_SMD:R_0805_2012Metric_Pad1.15x1.40mm_HandSolder, B.Cu at (229.8, 94.1)
- added RL49: R, Resistor_SMD:R_0805_2012Metric_Pad1.15x1.40mm_HandSolder, B.Cu at (238.5, 111.8)
- added RL5: R, Resistor_SMD:R_0805_2012Metric_Pad1.15x1.40mm_HandSolder, B.Cu at (54.4, 125.7)
- added RL50: R, Resistor_SMD:R_0805_2012Metric_Pad1.15x1.40mm_HandSolder, B.Cu at (247.0, 129.4)
- added RL51: R, Resistor_SMD:R_0805_2012Metric_Pad1.15x1.40mm_HandSolder, B.Cu at (239.4, 48.4)
- added RL52: R, Resistor_SMD:R_0805_2012Metric_Pad1.15x1.40mm_HandSolder, B.Cu at (235.0, 73.5)
- added RL53: R, Resistor_SMD:R_0805_2012Metric_Pad1.15x1.40mm_HandSolder, B.Cu at (248.5, 90.2)
- added RL54: R, Resistor_SMD:R_0805_2012Metric_Pad1.15x1.40mm_HandSolder, B.Cu at (257.1, 107.8)
- added RL55: R, Resistor_SMD:R_0805_2012Metric_Pad1.15x1.40mm_HandSolder, B.Cu at (265.7, 125.4)
- added RL56: R, Resistor_SMD:R_0805_2012Metric_Pad1.15x1.40mm_HandSolder, B.Cu at (260.3, 146.0)
- added RL57: R, Resistor_SMD:R_0805_2012Metric_Pad1.15x1.40mm_HandSolder, B.Cu at (258.1, 44.5)
- added RL58: R, Resistor_SMD:R_0805_2012Metric_Pad1.15x1.40mm_HandSolder, B.Cu at (253.8, 69.6)
- added RL59: R, Resistor_SMD:R_0805_2012Metric_Pad1.15x1.40mm_HandSolder, B.Cu at (266.9, 86.2)
- added RL6: R, Resistor_SMD:R_0805_2012Metric_Pad1.15x1.40mm_HandSolder, B.Cu at (47.0, 144.8)
- added RL60: R, Resistor_SMD:R_0805_2012Metric_Pad1.15x1.40mm_HandSolder, B.Cu at (276.6, 106.5)
- added RL61: R, Resistor_SMD:R_0805_2012Metric_Pad1.15x1.40mm_HandSolder, B.Cu at (286.0, 125.6)
- added RL62: R, Resistor_SMD:R_0805_2012Metric_Pad1.15x1.40mm_HandSolder, B.Cu at (277.9, 43.2)
- added RL63: R, Resistor_SMD:R_0805_2012Metric_Pad1.15x1.40mm_HandSolder, B.Cu at (272.9, 66.9)
- added RL64: R, Resistor_SMD:R_0805_2012Metric_Pad1.15x1.40mm_HandSolder, B.Cu at (286.5, 87.5)
- added RL65: R, Resistor_SMD:R_0805_2012Metric_Pad1.15x1.40mm_HandSolder, B.Cu at (295.7, 106.6)
- added RL66: R, Resistor_SMD:R_0805_2012Metric_Pad1.15x1.40mm_HandSolder, B.Cu at (312.3, 125.6)
- added RL67: R, Resistor_SMD:R_0805_2012Metric_Pad1.15x1.40mm_HandSolder, B.Cu at (296.9, 43.2)
- added RL68: R, Resistor_SMD:R_0805_2012Metric_Pad1.15x1.40mm_HandSolder, B.Cu at (291.8, 68.4)
- added RL69: R, Resistor_SMD:R_0805_2012Metric_Pad1.15x1.40mm_HandSolder, B.Cu at (305.6, 87.5)
- added RL7: R, Resistor_SMD:R_0805_2012Metric_Pad1.15x1.40mm_HandSolder, B.Cu at (68.6, 43.2)
- added RL70: R, Resistor_SMD:R_0805_2012Metric_Pad1.15x1.40mm_HandSolder, B.Cu at (326.5, 106.5)
- added RL71: R, Resistor_SMD:R_0805_2012Metric_Pad1.15x1.40mm_HandSolder, B.Cu at (324.2, 149.5)
- added RL72: R, Resistor_SMD:R_0805_2012Metric_Pad1.15x1.40mm_HandSolder, B.Cu at (323.6, 44.7)
- added RL73: R, Resistor_SMD:R_0805_2012Metric_Pad1.15x1.40mm_HandSolder, B.Cu at (310.9, 68.6)
- added RL74: R, Resistor_SMD:R_0805_2012Metric_Pad1.15x1.40mm_HandSolder, B.Cu at (329.4, 87.5)
- added RL75: R, Resistor_SMD:R_0805_2012Metric_Pad1.15x1.40mm_HandSolder, B.Cu at (343.3, 130.4)
- added RL76: R, Resistor_SMD:R_0805_2012Metric_Pad1.15x1.40mm_HandSolder, B.Cu at (343.2, 149.5)
- added RL77: R, Resistor_SMD:R_0805_2012Metric_Pad1.15x1.40mm_HandSolder, B.Cu at (349.6, 44.7)
- added RL78: R, Resistor_SMD:R_0805_2012Metric_Pad1.15x1.40mm_HandSolder, B.Cu at (329.9, 68.6)
- added RL79: R, Resistor_SMD:R_0805_2012Metric_Pad1.15x1.40mm_HandSolder, B.Cu at (353.8, 63.7)
- added RL8: R, Resistor_SMD:R_0805_2012Metric_Pad1.15x1.40mm_HandSolder, B.Cu at (73.7, 68.6)
- added RL80: R, Resistor_SMD:R_0805_2012Metric_Pad1.15x1.40mm_HandSolder, B.Cu at (358.0, 82.8)
- added RL81: R, Resistor_SMD:R_0805_2012Metric_Pad1.15x1.40mm_HandSolder, B.Cu at (362.2, 101.8)
- added RL82: R, Resistor_SMD:R_0805_2012Metric_Pad1.15x1.40mm_HandSolder, B.Cu at (362.3, 149.5)
- added RL9: R, Resistor_SMD:R_0805_2012Metric_Pad1.15x1.40mm_HandSolder, B.Cu at (79.2, 87.6)
- D1, D10, D11, D12, D13, D14, D15, D16, D17, D18, D19, D2, D20, D21, D22, D23, D24, D25, D26, D27, D28, D29, D3, D30, D31, D32, D33, D34, D35, D36, D37, D38, D39, D4, D40, D41, D42, D43, D44, D45, D46, D47, D48, D49, D5, D50, D51, D52, D53, D54, D55, D56, D57, D58, D59, D6, D60, D61, D62, D63, D64, D65, D66, D67, D7, D8, D9: footprint Diodes_SMD:D_SOD-123 -> Diode_SMD:D_SOD-123
- J1: value USB_B_Micro -> USB_B_Mini; footprint Connectors_USB:USB_Micro-B_Molex-105017-0001 -> Keebio-Parts:USB-Mini-B_2leg
- R1, R2, R3, R4: footprint Resistors_SMD:R_0805_HandSoldering -> Resistor_SMD:R_0805_2012Metric_Pad1.15x1.40mm_HandSolder
- moved D67 101.7 mm to (297.0, 37.8)
- moved D62 101.7 mm to (277.9, 37.8)
- moved D6 98.2 mm to (47.1, 139.3)
- moved D34 89.4 mm to (166.7, 157.1), turned to 78 degrees
- moved D56 86.9 mm to (259.2, 140.7), turned to 102 degrees
- moved D58 84.9 mm to (252.7, 64.4), turned to 102 degrees
- moved D33 82.3 mm to (161.4, 135.8), turned to 78 degrees
- moved D46 82.0 mm to (215.1, 47.9)
- moved D23 81.8 mm to (127.0, 46.2)
- moved D55 79.4 mm to (264.6, 120.1), turned to 102 degrees
- moved D57 72.1 mm to (257.0, 39.1), turned to 102 degrees
- moved D64 72.0 mm to (286.5, 82.1)
- moved D65 68.2 mm to (295.6, 101.1)
- moved D18 63.3 mm to (108.4, 42.2)
- moved D39 62.4 mm to (208.6, 131.9)
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- renumbered VCC to J12, D+ to J13, D- to J14, GND to J15, MISO to J2, VCC to J3, SCK to J4, MOSI to J5, RES to J6, GND to J7, PF4 to J8, PF5 to J9
Connections:
- D10 pad 1: /row0 -> /row3
- D11 pad 1: /row1 -> /row4
- D12 pad 1: /row2 -> /row0
- D13 pad 1: /row3 -> /row1
- D14 pad 1: /row4 -> /row2
- D15 pad 1: /row0 -> /row3
- D16 pad 1: /row1 -> /row4
- D17 pad 1: /row2 -> /row5
- D18 pad 1: /row3 -> /row0
- D19 pad 1: /row0 -> /row1
- D20 pad 1: /row1 -> /row2
- D21 pad 1: /row2 -> /row3
- D22 pad 1: /row3 -> /row4
- D23 pad 1: /row4 -> /row0
- D24 pad 1: /row0 -> /row1
- D25 pad 1: /row1 -> /row2
- D26 pad 1: /row2 -> /row3
- D27 pad 1: /row3 -> /row4
- D28 pad 1: /row4 -> /row5
- D33 pad 1: /row0 -> /row4
- D34 pad 1: /row1 -> /row5
- D35 pad 1: /row2 -> /row0
- D36 pad 1: /row3 -> /row1
- D37 pad 1: /row4 -> /row2
- D38 pad 1: /row0 -> /row3
- D39 pad 1: /row1 -> /row4
- D40 pad 1: /row2 -> /row0
- D41 pad 1: /row3 -> /row1
- D42 pad 1: /row0 -> /row2
- D43 pad 1: /row1 -> /row3
- D44 pad 1: /row2 -> /row4
- D45 pad 1: /row3 -> /row5
- D46 pad 1: /row4 -> /row0
- D47 pad 1: /row0 -> /row1
- D48 pad 1: /row1 -> /row2
- D49 pad 1: /row2 -> /row3
- D50 pad 1: /row3 -> /row4
- D55 pad 1: /row0 -> /row4
- D56 pad 1: /row1 -> /row5
- D57 pad 1: /row2 -> /row0
- D58 pad 1: /row4 -> /row1
- D59 pad 1: /row0 -> /row2
- D6 pad 1: /row0 -> /row5
- D60 pad 1: /row1 -> /row3
- D61 pad 1: /row3 -> /row4
- D62 pad 1: /row4 -> /row0
- D63 pad 1: /row0 -> /row1
- D64 pad 1: /row1 -> /row2
- D65 pad 1: /row2 -> /row3
- D66 pad 1: /row3 -> /row4
- D67 pad 1: /row4 -> /row0
- D7 pad 1: /row1 -> /row0
- D8 pad 1: /row2 -> /row1
- D9 pad 1: /row3 -> /row2
- U2 pad 36: /PF7 -> /row5
- U2 pad 37: /PF6 -> Net-(R5-Pad1)
Routing:
- net /row4: track 433.8 -> 14.5 mm, vias 2 -> 1
- net /row3: track 432.5 -> 15.6 mm, vias 2 -> 1
- net /row2: track 399.4 -> 17.3 mm, vias 4 -> 1
- net /row1: track 384.1 -> 24.2 mm, vias 4 -> 1
- net /row0: track 328.0 -> 27.6 mm, vias 4 -> 1
- net /col13: track 269.0 -> 0.00 mm
- net /col12: track 249.0 -> 0.00 mm
- net /col11: track 230.6 -> 0.00 mm
- net /MISO: track 272.2 -> 46.0 mm
- net /col10: track 221.3 -> 0.00 mm
- net /col0: track 204.4 -> 23.8 mm
- net /col2: track 175.7 -> 26.6 mm
- net /col1: track 166.8 -> 24.1 mm
- net /col4: track 135.2 -> 6.23 mm
- net /col3: track 133.3 -> 6.39 mm
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- removed copper zone on F.Cu, net GND
Other:
- board size 339.1 x 118.7 mm -> 339.1 x 143.2 mm
- board text removed: "Fate Design Rev 1.1"

Commit message: added column and row routing
Parts:
- MX28: footprint ai03-MX_only:MXOnly-2U-FLIPPED-ReversedStabilizers -> ai03-MX_only:MXOnly-2U-ReversedStabilizers
- MX70: footprint ai03-MX_only:MXOnly-2.25U-FLIPPED-ReversedStabilizers -> ai03-MX_only:MXOnly-2.25U-ReversedStabilizers
Routing:
- net /ledGND: track 10.9 -> 139.5 mm
- net /row0: track 27.6 -> 75.9 mm
- net Net-(D4-Pad2): track 0.00 -> 11.0 mm
- net /SCK: track 72.3 -> 62.3 mm
- net Net-(D13-Pad2): track 0.00 -> 7.21 mm
- net Net-(MX24-Pad4): track 0.00 -> 7.16 mm
- net Net-(MX25-Pad4): track 0.00 -> 7.13 mm
- net Net-(MX14-Pad4): track 0.00 -> 7.11 mm
- net Net-(MX31-Pad4): track 0.00 -> 7.10 mm
- net Net-(MX18-Pad4): track 0.00 -> 7.09 mm
- net Net-(MX23-Pad4): track 0.00 -> 7.07 mm
- net Net-(MX36-Pad4): track 0.00 -> 7.06 mm
- net Net-(MX29-Pad4): track 0.00 -> 7.04 mm
- net Net-(MX34-Pad4): track 0.00 -> 7.02 mm
- net Net-(MX30-Pad4): track 0.00 -> 6.96 mm
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
Commit message: added matrix routing
Parts:
- moved H4 24.5 mm to (111.8, 145.0)
- moved H1 24.4 mm to (56.9, 72.6)
- moved H8 24.3 mm to (345.4, 134.5)
- moved H2 16.4 mm to (52.3, 139.6)
- moved H7 7.61 mm to (337.1, 48.8)
- moved H6 5.45 mm to (240.7, 144.5)
Routing:
- net +5V: track 0.00 -> 1745.8 mm
- net /ledGND: track 139.5 -> 1862.0 mm, vias 1 -> 3
- net /row5: track 18.7 -> 468.7 mm, vias 0 -> 2
- net /row4: track 14.5 -> 458.6 mm, vias 1 -> 2
- net /row3: track 15.6 -> 420.9 mm, vias 1 -> 2
- net /row2: track 17.3 -> 400.3 mm, vias 1 -> 2
- net /row1: track 24.2 -> 322.9 mm, vias 1 -> 2
- net /row0: track 75.9 -> 366.8 mm, vias 1 -> 4
- net /MISO: track 46.0 -> 328.8 mm
- net /col13: track 0.00 -> 268.0 mm
- net /col12: track 0.00 -> 251.4 mm
- net /col0: track 23.8 -> 259.7 mm
- net /col11: track 0.00 -> 206.0 mm
- net /col2: track 26.6 -> 219.4 mm, vias 2 -> 3
- net /col1: track 24.1 -> 209.0 mm
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
Commit message: finished pcb v2
Parts:
- added  G2: LOGO, adelheid:adelheid-logo, B.Cu at (286.8, 139.1)
- added G1: LOGO, adelheid:adelheid-logo, F.Cu at (286.8, 142.6)
- added LS1: LED, LED_SMD:LED_0805_2012Metric_Pad1.15x1.40mm_HandSolder, B.Cu at (27.9, 39.1)
- added LS10: LED, LED_SMD:LED_0805_2012Metric_Pad1.15x1.40mm_HandSolder, B.Cu at (361.9, 137.2)
- added LS11: LED, LED_SMD:LED_0805_2012Metric_Pad1.15x1.40mm_HandSolder, B.Cu at (361.9, 86.4)
- added LS12: LED, LED_SMD:LED_0805_2012Metric_Pad1.15x1.40mm_HandSolder, B.Cu at (361.9, 39.1)
- added LS13: LED, LED_SMD:LED_0805_2012Metric_Pad1.15x1.40mm_HandSolder, B.Cu at (237.2, 26.9)
- added LS14: LED, LED_SMD:LED_0805_2012Metric_Pad1.15x1.40mm_HandSolder, B.Cu at (281.4, 26.9)
- added LS15: LED, LED_SMD:LED_0805_2012Metric_Pad1.15x1.40mm_HandSolder, B.Cu at (331.7, 27.2)
- added LS16: LED, LED_SMD:LED_0805_2012Metric_Pad1.15x1.40mm_HandSolder, B.Cu at (131.1, 26.9)
- added LS17: LED, LED_SMD:LED_0805_2012Metric_Pad1.15x1.40mm_HandSolder, B.Cu at (67.3, 26.9)
- added LS2: LED, LED_SMD:LED_0805_2012Metric_Pad1.15x1.40mm_HandSolder, B.Cu at (27.9, 86.4)
- added LS3: LED, LED_SMD:LED_0805_2012Metric_Pad1.15x1.40mm_HandSolder, B.Cu at (27.9, 135.6)
- added LS4: LED, LED_SMD:LED_0805_2012Metric_Pad1.15x1.40mm_HandSolder, B.Cu at (56.4, 151.1)
- added LS5: LED, LED_SMD:LED_0805_2012Metric_Pad1.15x1.40mm_HandSolder, B.Cu at (127.8, 156.5)
- added LS6: LED, LED_SMD:LED_0805_2012Metric_Pad1.15x1.40mm_HandSolder, B.Cu at (175.7, 165.1)
- added LS7: LED, LED_SMD:LED_0805_2012Metric_Pad1.15x1.40mm_HandSolder, B.Cu at (211.6, 159.0)
- added LS8: LED, LED_SMD:LED_0805_2012Metric_Pad1.15x1.40mm_HandSolder, B.Cu at (271.8, 151.1)
- added LS9: LED, LED_SMD:LED_0805_2012Metric_Pad1.15x1.40mm_HandSolder, B.Cu at (328.2, 151.1)
- added RS1: R, Resistor_SMD:R_0805_2012Metric_Pad1.15x1.40mm_HandSolder, B.Cu at (29.0, 43.4)
- added RS10: R, Resistor_SMD:R_0805_2012Metric_Pad1.15x1.40mm_HandSolder, B.Cu at (360.9, 132.8)
- added RS11: R, Resistor_SMD:R_0805_2012Metric_Pad1.15x1.40mm_HandSolder, B.Cu at (360.9, 82.0)
- added RS12: R, Resistor_SMD:R_0805_2012Metric_Pad1.15x1.40mm_HandSolder, B.Cu at (360.9, 34.8)
- added RS13: R, Resistor_SMD:R_0805_2012Metric_Pad1.15x1.40mm_HandSolder, B.Cu at (232.9, 27.9)
- added RS14: R, Resistor_SMD:R_0805_2012Metric_Pad1.15x1.40mm_HandSolder, B.Cu at (277.4, 27.9)
- added RS15: R, Resistor_SMD:R_0805_2012Metric_Pad1.15x1.40mm_HandSolder, B.Cu at (327.4, 28.2)
- added RS16: R, Resistor_SMD:R_0805_2012Metric_Pad1.15x1.40mm_HandSolder, B.Cu at (126.7, 27.9)
- added RS17: R, Resistor_SMD:R_0805_2012Metric_Pad1.15x1.40mm_HandSolder, B.Cu at (63.0, 27.9)
- added RS2: R, Resistor_SMD:R_0805_2012Metric_Pad1.15x1.40mm_HandSolder, B.Cu at (29.0, 90.7)
- added RS3: R, Resistor_SMD:R_0805_2012Metric_Pad1.15x1.40mm_HandSolder, B.Cu at (29.0, 140.0)
- added RS4: R, Resistor_SMD:R_0805_2012Metric_Pad1.15x1.40mm_HandSolder, B.Cu at (60.7, 150.1)
- added RS5: R, Resistor_SMD:R_0805_2012Metric_Pad1.15x1.40mm_HandSolder, B.Cu at (131.8, 157.3)
- added RS6: R, Resistor_SMD:R_0805_2012Metric_Pad1.15x1.40mm_HandSolder, B.Cu at (175.7, 161.8)
- added RS7: R, Resistor_SMD:R_0805_2012Metric_Pad1.15x1.40mm_HandSolder, B.Cu at (215.9, 158.0)
- added RS8: R, Resistor_SMD:R_0805_2012Metric_Pad1.15x1.40mm_HandSolder, B.Cu at (276.1, 150.1)
- added RS9: R, Resistor_SMD:R_0805_2012Metric_Pad1.15x1.40mm_HandSolder, B.Cu at (332.2, 150.1)
- moved RL82 12.4 mm to (350.0, 148.3)
- moved D82 4.47 mm to (360.2, 147.8)
- moved D81 4.32 mm to (360.0, 92.7)
- moved RL81 2.67 mm to (359.9, 100.5)
Connections:
- MX1 pad 3: +5V -> VCC
- MX10 pad 3: +5V -> VCC
- MX11 pad 3: +5V -> VCC
- MX12 pad 3: +5V -> VCC
- MX13 pad 3: +5V -> VCC
- MX14 pad 3: +5V -> VCC
- MX15 pad 3: +5V -> VCC
- MX16 pad 3: +5V -> VCC
- MX17 pad 3: +5V -> VCC
- MX18 pad 3: +5V -> VCC
- MX19 pad 3: +5V -> VCC
- MX2 pad 3: +5V -> VCC
- MX20 pad 3: +5V -> VCC
- MX21 pad 3: +5V -> VCC
- MX22 pad 3: +5V -> VCC
- MX23 pad 3: +5V -> VCC
- MX24 pad 3: +5V -> VCC
- MX25 pad 3: +5V -> VCC
- MX26 pad 3: +5V -> VCC
- MX27 pad 3: +5V -> VCC
- MX28 pad 3: +5V -> VCC
- MX29 pad 3: +5V -> VCC
- MX3 pad 3: +5V -> VCC
- MX30 pad 3: +5V -> VCC
- MX31 pad 3: +5V -> VCC
- MX32 pad 3: +5V -> VCC
- MX33 pad 3: +5V -> VCC
- MX34 pad 3: +5V -> VCC
- MX35 pad 3: +5V -> VCC
- MX36 pad 3: +5V -> VCC
- MX37 pad 3: +5V -> VCC
- MX38 pad 3: +5V -> VCC
- MX39 pad 3: +5V -> VCC
- MX4 pad 3: +5V -> VCC
- MX40 pad 3: +5V -> VCC
- MX41 pad 3: +5V -> VCC
- MX42 pad 3: +5V -> VCC
- MX43 pad 3: +5V -> VCC
- MX44 pad 3: +5V -> VCC
- MX45 pad 3: +5V -> VCC
- MX46 pad 3: +5V -> VCC
- MX47 pad 3: +5V -> VCC
- MX48 pad 3: +5V -> VCC
- MX49 pad 3: +5V -> VCC
- MX4_1 pad 3: +5V -> VCC
- MX5 pad 3: +5V -> VCC
- MX50 pad 3: +5V -> VCC
- MX51 pad 3: +5V -> VCC
- MX52 pad 3: +5V -> VCC
- MX53 pad 3: +5V -> VCC
- MX54 pad 3: +5V -> VCC
- MX55 pad 3: +5V -> VCC
- MX56 pad 3: +5V -> VCC
- MX57 pad 3: +5V -> VCC
- MX58 pad 3: +5V -> VCC
- MX59 pad 3: +5V -> VCC
- MX6 pad 3: +5V -> VCC
- MX60 pad 3: +5V -> VCC
- MX61 pad 3: +5V -> VCC
- MX62 pad 3: +5V -> VCC
- MX63 pad 3: +5V -> VCC
- MX64 pad 3: +5V -> VCC
- MX65 pad 3: +5V -> VCC
- MX66 pad 3: +5V -> VCC
- MX67 pad 3: +5V -> VCC
- MX68 pad 3: +5V -> VCC
- MX69 pad 3: +5V -> VCC
- MX7 pad 3: +5V -> VCC
- MX70 pad 3: +5V -> VCC
- MX71 pad 3: +5V -> VCC
- MX72 pad 3: +5V -> VCC
- MX73 pad 3: +5V -> VCC
- MX74 pad 3: +5V -> VCC
- MX75 pad 3: +5V -> VCC
- MX76 pad 3: +5V -> VCC
- MX77 pad 3: +5V -> VCC
- MX78 pad 3: +5V -> VCC
- MX79 pad 3: +5V -> VCC
- MX8 pad 3: +5V -> VCC
- MX80 pad 3: +5V -> VCC
- MX81 pad 3: +5V -> VCC
- MX82 pad 3: +5V -> VCC
- MX9 pad 3: +5V -> VCC
Routing:
- net VCC: track 205.4 -> 2646.7 mm, vias 9 -> 15
- net +5V: track 1745.8 -> 0.00 mm
- net /ledGND: track 1862.0 -> 2409.6 mm, vias 3 -> 19
- net /row1: track 322.9 -> 347.7 mm
- net /row5: track 468.7 -> 480.6 mm
- net GND: track 71.6 -> 61.7 mm, vias 12 -> 19
- net Net-(J1-Pad2): track 45.1 -> 40.8 mm, vias 0 -> 1
- net Net-(LS4-Pad1): track 0.00 -> 3.30 mm
- net Net-(LS6-Pad1): track 0.00 -> 3.30 mm
- net Net-(LS11-Pad1): track 0.00 -> 3.30 mm
- net Net-(LS10-Pad1): track 0.00 -> 3.30 mm
- net Net-(LS8-Pad1): track 0.00 -> 3.30 mm
- net Net-(LS17-Pad1): track 0.00 -> 3.29 mm
- net Net-(LS12-Pad1): track 0.00 -> 3.29 mm
- net Net-(LS16-Pad1): track 0.00 -> 3.29 mm
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- added copper zone on F.Cu, net GND
Other:
- board text added: "."
- board text added: "fork of FateNozomi/Arisu by floookay [v2]"
